File: grogu-dib-board.kicad_sch (KiCad schematic)
At the start: 4 parts, among them J1 ERF8-050-05.0-L-DV-K-TR, J2 ERF8-050-05.0-L-DV-K-TR

Commit message: schematic done
Parts:
- removed H1: MountingHole, symbol Mechanical:MountingHole
- renumbered U1 to J3
Connections:
- net FB2.DVML.MUX: now also J3.E38
- net FB2.HF1: now also J1.01
- net FB2.HF2: now also J1.21
- net FB2.HF3: now also J1.25
- net FB2.HF5: now also J1.63; no longer J1.69
- net FB2.LF: now also J1.07, J1.15, J1.23, J1.31, J1.49, J3.F1, J3.F14, J3.F16, J3.F18, J3.F23, J3.F25, J3.F27, J3.F36, J3.F5, J3.F7, J3.F9
- net FB2.MFD.N: now also J1.51
- net FB2.MFDCLK.N: now also J1.55
- net FB2.MLD.N: now also J1.33
- net FB2.MLDCLK.N: now also J1.37; no longer J1.39
- net FB2.PREF.HS: now also J1.67
- net FB3.LF: now also J3.B16, J3.B18, J3.B20, J3.B25, J3.B27, J3.B29, J3.B34, J3.B36, J3.B38, J3.B42, J3.B7
- net FB4.HF1: now reaches J3.A46
- net FB4.HF1: now also J2.80
- net FB4.DVMH: now reaches J3.A48
- net FB4.DVMH: now also J2.70
- net FB4.DVML: now reaches J3.A50
- net FB4.DVML: now also J2.68
- net FB4.LF: now reaches J3.A52
- net FB4.LF: now also J2.02, J2.32, J2.40, J2.50, J2.58, J2.66, J2.74, J3.A61, J3.A63, J3.A65, J3.A70, J3.A72, J3.A74, J3.A79, J3.A81, J3.A83, J3.A87, J3.B52, J3.B61, J3.B63, J3.B65, J3.B70, J3.B72, J3.B74, J3.B79, J3.B81, J3.B83, J3.B87
- net FB4.HF2: now reaches J3.A54
- net FB4.HF2: now also J2.60
- net FB4.HF3: now reaches J3.A59
- net FB4.HF3: now also J2.56
- net FB4.MLD.N: now reaches J3.A62
- net FB4.MLD.N: now also J2.48
- net FB4.MLDCLK.N: now reaches J3.A64
- net FB4.MLDCLK.N: now also J2.44
- net FB4.HF4: now reaches J3.A68
- net FB4.HF4: now also J2.38
- net FB4.MFD.N: now reaches J3.A71
- net FB4.MFD.N: now also J2.30
- net FB4.MFDCLK.N: now reaches J3.A73
- net FB4.MFDCLK.N: now also J2.26
- net FB4.HF5: now reaches J3.A76
- net FB4.HF5: now also J2.18
- net FB4.PREF.HS: now reaches J3.A80
- net FB4.PREF.HS: now also J2.14
- net FB4.PREF.F: now reaches J3.A82
- net FB4.PREF.F: now also J2.10
- net FB4.HF6: now reaches J3.A85
- net FB4.HF6: now also J2.08
- net FB3.HS1: now reaches J3.B1
- net FB3.HS1: now also J1.78
- net FB3.HS3: now reaches J3.B14
- net FB3.HS3: now also J1.54
- net FB3.MLD.P: now reaches J3.B17
- net FB3.MLD.P: now also J1.46
- net FB3.MLDCLK.P: now reaches J3.B19
- net FB3.MLDCLK.P: now also J1.42
- net FB3.HS4: now reaches J3.B23
- net FB3.HS4: now also J1.36
- net FB3.MFD.P: now reaches J3.B26
- net FB3.MFD.P: now also J1.28
- net FB3.MFDCLK.P: now reaches J3.B28
- net FB3.MFDCLK.P: now also J1.24
- net FB3.HS5: now reaches J3.B31
- net FB3.HS5: now also J1.20
- net FB3.PREF.LS: now reaches J3.B35
- net FB3.PREF.LS: now also J1.16
- net FB3.PREF.G: now reaches J3.B37
- net FB3.PREF.G: now also J1.12
- net FB3.HS6: now reaches J3.B40
- net FB3.HS6: now also J1.06
- net FB4.HS1: now reaches J3.B46
- net FB4.HS1: now also J2.78
- net FB4.HS2: now reaches J3.B54
- net FB4.HS2: now also J2.62
- net FB4.HS3: now reaches J3.B59
- net FB4.HS3: now also J2.54
- net FB4.MLD.P: now reaches J3.B62
- net FB4.MLD.P: now also J2.46
- net FB4.MLDCLK.P: now reaches J3.B64
- net FB4.MLDCLK.P: now also J2.42
- net FB4.HS4: now reaches J3.B68
- net FB4.HS4: now also J2.36
- net FB4.MFD.P: now reaches J3.B71
- net FB4.MFD.P: now also J2.28
- net FB4.MFDCLK.P: now reaches J3.B73
- net FB4.MFDCLK.P: now also J2.24
- net FB4.HS5: now reaches J3.B76
- net FB4.HS5: now also J2.20
- net FB4.PREF.LS: now reaches J3.B80
- net FB4.PREF.LS: now also J2.16
- net FB4.PREF.G: now reaches J3.B82
- net FB4.PREF.G: now also J2.12
- net FB4.HS6: now reaches J3.B85
- net FB4.HS6: now also J2.06
- net FB3.HS2: now reaches J3.B9
- net FB3.HS2: now also J1.62
- net FB3.LS3: now reaches J3.C16
- net FB3.LS3: now also J1.52
- net FB3.LS4: now reaches J3.C25
- net FB3.LS4: now also J1.34
- net FB3.LS5: now reaches J3.C29
- net FB3.LS5: now also J1.22
- net FB3.LS1: now reaches J3.C3
- net FB3.LS1: now also J1.76
- net FB3.LS6: now reaches J3.C42
- net FB3.LS6: now also J1.04
- net FB4.LS1: now reaches J3.C48
- net FB4.LS1: now also J2.76
- net FB3.DVML.MUX: now reaches J3.C5
- net FB3.DVML.MUX: now also J1.72
- net FB4.DVML.MUX: now reaches J3.C50
- net FB4.DVML.MUX: now also J2.72
- net FB4.LS2: now reaches J3.C52
- net FB4.LS2: now also J2.64
- net FB4.LS3: now reaches J3.C61
- net FB4.LS3: now also J2.52
- net FB3.LS2: now reaches J3.C7
- net FB3.LS2: now also J1.64
- net FB4.LS4: now reaches J3.C70
- net FB4.LS4: now also J2.34
- net FB4.LS5: now reaches J3.C74
- net FB4.LS5: now also J2.22
- net FB4.LS6: now reaches J3.C87
- net FB4.LS6: now also J2.04
- net FB2.LS6: now reaches J3.E1
- net FB2.LS6: now also J1.77
- net FB2.LS5: now reaches J3.E14
- net FB2.LS5: now also J1.59
- net FB2.LS4: now reaches J3.E18
- net FB2.LS4: now also J1.47
- net FB2.LS3: now reaches J3.E27
- net FB2.LS3: now also J1.29
- net FB2.LS2: now reaches J3.E36
- net FB2.LS2: now also J1.17
- net FB2.LS1: now reaches J3.E40
- net FB2.LS1: now also J1.05
- net FB1.LS6: now reaches J3.E46
- net FB1.LS6: now also J2.77
- net FB1.LS5: now reaches J3.E59
- net FB1.LS5: now also J2.59
- net FB1.LS4: now reaches J3.E63
- net FB1.LS4: now also J2.47
- net FB1.LS3: now reaches J3.E72
- net FB1.LS3: now also J2.29
- net FB1.LS2: now reaches J3.E81
- net FB1.LS2: now also J2.17
- net FB1.DVML.MUX: now reaches J3.E83
- net FB1.DVML.MUX: now also J2.09
- net FB1.LS1: now reaches J3.E85
- net FB1.LS1: now also J2.05
- net FB2.HS5: now reaches J3.F12
- net FB2.HS5: now also J1.61
- net FB2.MFDCLK.P: now reaches J3.F15
- net FB2.MFDCLK.P: now also J1.57
- net FB2.MFD.P: now reaches J3.F17
- net FB2.MFD.P: now also J1.53
- net FB2.HS4: now reaches J3.F20
- net FB2.HS4: now also J1.45
- net FB2.MLDCLK.P: now reaches J3.F24
- net FB2.MLDCLK.P: now also J1.39
- net FB2.MLD.P: now reaches J3.F26
- net FB2.MLD.P: now also J1.35
- net FB2.HS3: now reaches J3.F29
- net FB2.HS3: now also J1.27
- net FB2.HS6: now reaches J3.F3
- net FB2.HS6: now also J1.75
- net FB2.HS2: now reaches J3.F34
- net FB2.HS2: now also J1.19
- net FB2.HS1: now reaches J3.F42
- net FB2.HS1: now also J1.03
- net FB1.LF: now reaches J3.F46
- net FB1.LF: now also J2.07, J2.15, J2.23, J2.31, J2.41, J2.49, J2.79, J3.F50, J3.F52, J3.F54, J3.F59, J3.F61, J3.F63, J3.F68, J3.F70, J3.F72, J3.F81, J3.G46, J3.G50, J3.G52, J3.G54, J3.G59, J3.G61, J3.G63, J3.G68, J3.G70, J3.G72, J3.G81
- net FB1.HS6: now reaches J3.F48
- net FB1.HS6: now also J2.75
- net FB1.PREF.G: now reaches J3.F51
- net FB1.PREF.G: now also J2.69
- net FB1.PREF.LS: now reaches J3.F53
- net FB1.PREF.LS: now also J2.65
- net FB1.HS5: now reaches J3.F57
- net FB1.HS5: now also J2.61
- net FB2.PREF.G: now reaches J3.F6
- net FB2.PREF.G: now also J1.69
- net FB1.MFDCLK.P: now reaches J3.F60
- net FB1.MFDCLK.P: now also J2.57
- net FB1.MFD.P: now reaches J3.F62
- net FB1.MFD.P: now also J2.53
- net FB1.HS4: now reaches J3.F65
- net FB1.HS4: now also J2.45
- net FB1.MLDCLK.P: now reaches J3.F69
- net FB1.MLDCLK.P: now also J2.39
- net FB1.MLD.P: now reaches J3.F71
- net FB1.MLD.P: now also J2.35
- net FB1.HS3: now reaches J3.F74
- net FB1.HS3: now also J2.27
- net FB1.HS2: now reaches J3.F79
- net FB1.HS2: now also J2.19
- net FB2.PREF.LS: now reaches J3.F8
- net FB2.PREF.LS: now also J1.65
- net FB1.HS1: now reaches J3.F87
- net FB1.HS1: now also J2.03
- net FB1.HF6: now reaches J3.G48
- net FB1.HF6: now also J2.73
- net FB1.PREF.F: now reaches J3.G51
- net FB1.PREF.F: now also J2.71
- net FB1.PREF.HS: now reaches J3.G53
- net FB1.PREF.HS: now also J2.67
- net FB1.HF5: now reaches J3.G57
- net FB1.HF5: now also J2.63
- net FB1.MFDCLK.N: now reaches J3.G60
- net FB1.MFDCLK.N: now also J2.55
- net FB1.MFD.N: now reaches J3.G62
- net FB1.MFD.N: now also J2.51
- net FB1.HF4: now reaches J3.G65
- net FB1.HF4: now also J2.43
- net FB1.MLDCLK.N: now reaches J3.G69
- net FB1.MLDCLK.N: now also J2.37
- net FB1.MLD.N: now reaches J3.G71
- net FB1.MLD.N: now also J2.33
- net FB1.HF3: now reaches J3.G74
- net FB1.HF3: now also J2.25
- net FB1.HF2: now reaches J3.G79
- net FB1.HF2: now also J2.21
- net FB1.DVML: now reaches J3.G83
- net FB1.DVML: now also J2.13
- net FB1.DVMH: now reaches J3.G85
- net FB1.DVMH: now also J2.11
- net FB1.HF1: now reaches J3.G87
- net FB1.HF1: now also J2.01
Other:
- moved on the sheet: J2
