File: grogu-dib-board.kicad_pcb (KiCad board)
At the start: 2 copper layers, 9.5 x 102.4 mm, 18 parts, among them J1 ERF8-050-05.0-L-DV-K-TR, J2 ERF8-050-05.0-L-DV-K-TR

Commit message: Summit Modifications
- Removed pads where connector hole emerges on bottom side
- Re-routed traces to avoid counterbore
- Soldermask clearance increased on bottom side for counterbore
- Removed stackup table (2mm thickness per summit quote)
Routing:
- net /FB3.PREF.F: track 8.99 -> 23.7 mm
- net /FB2.DVMH: track 12.9 -> 18.8 mm, vias 1 -> 2

Commit message: Fabrication Outputs for Summit Revisions
Other:
- board text removed: "0"
- board text removed: "0 in"
- board text removed: "0.0003937007874 in"
- board text removed: "0.001377952756 in"
- board text removed: "0.02"
- board text removed: "0.07145669291 in"
- board text removed: "1"
- board text removed: "3.3"
- board text removed: "4.5"
- board text removed: "B.Cu"
- board text removed: "B.Mask"
- board text removed: "B.Paste"
- board text removed: "B.Silkscreen"
- board text removed: "Bottom Silk Screen"
- board text removed: "Bottom Solder Mask"
- board text removed: "Bottom Solder Paste"
- board text removed: "Color"
- board text removed: "Dielectric 1"
- board text removed: "Epsilon R"
- board text removed: "F.Cu"
- board text removed: "F.Mask"
- board text removed: "F.Paste"
- board text removed: "F.Silkscreen"
- board text removed: "FR4"
- board text removed: "Layer Name"
- board text removed: "Loss Tangent"
- board text removed: "Material"
- board text removed: "Not specified"
- board text removed: "Thickness (inches)"
- board text removed: "Top Silk Screen"
- board text removed: "Top Solder Mask"
- board text removed: "Top Solder Paste"
- board text removed: "Type"
- board text removed: "copper"
- board text removed: "core"

Commit message: first pass routing
Parts:
- moved J2 0.15 mm to (73.5, 116.2)
- moved J1 0.11 mm to (73.5, 66.0)
- moved J3 0.08 mm to (73.7, 91.1)
- renumbered U1 to J3
Connections:
- J1 pad 01: unconnected-(J1-Pad01) -> /FB2.HF1
- J1 pad 03: unconnected-(J1-Pad03) -> /FB2.HS1
- J1 pad 04: unconnected-(J1-Pad04) -> /FB3.LS6
- J1 pad 05: unconnected-(J1-Pad05) -> /FB2.LS1
- J1 pad 06: unconnected-(J1-Pad06) -> /FB3.HS6
- J1 pad 07: unconnected-(J1-Pad07) -> /FB2.LF
- J1 pad 12: unconnected-(J1-Pad12) -> /FB3.PREF.G
- J1 pad 15: unconnected-(J1-Pad15) -> /FB2.LF
- J1 pad 16: unconnected-(J1-Pad16) -> /FB3.PREF.LS
- J1 pad 17: unconnected-(J1-Pad17) -> /FB2.LS2
- J1 pad 19: unconnected-(J1-Pad19) -> /FB2.HS2
- J1 pad 20: unconnected-(J1-Pad20) -> /FB3.HS5
- J1 pad 21: unconnected-(J1-Pad21) -> /FB2.HF2
- J1 pad 22: unconnected-(J1-Pad22) -> /FB3.LS5
- J1 pad 23: unconnected-(J1-Pad23) -> /FB2.LF
- J1 pad 24: unconnected-(J1-Pad24) -> /FB3.MFDCLK.P
- J1 pad 25: unconnected-(J1-Pad25) -> /FB2.HF3
- J1 pad 27: unconnected-(J1-Pad27) -> /FB2.HS3
- J1 pad 28: unconnected-(J1-Pad28) -> /FB3.MFD.P
- J1 pad 29: unconnected-(J1-Pad29) -> /FB2.LS3
- J1 pad 31: unconnected-(J1-Pad31) -> /FB2.LF
- J1 pad 33: unconnected-(J1-Pad33) -> /FB2.MLD.N
- J1 pad 34: unconnected-(J1-Pad34) -> /FB3.LS4
- J1 pad 35: unconnected-(J1-Pad35) -> /FB2.MLD.P
- J1 pad 36: unconnected-(J1-Pad36) -> /FB3.HS4
- J1 pad 37: unconnected-(J1-Pad37) -> /FB2.MLDCLK.N
- J1 pad 39: /FB2.MLDCLK.N -> /FB2.MLDCLK.P
- J1 pad 42: unconnected-(J1-Pad42) -> /FB3.MLDCLK.P
- J1 pad 45: unconnected-(J1-Pad45) -> /FB2.HS4
- J1 pad 46: unconnected-(J1-Pad46) -> /FB3.MLD.P
- J1 pad 47: unconnected-(J1-Pad47) -> /FB2.LS4
- J1 pad 49: unconnected-(J1-Pad49) -> /FB2.LF
- J1 pad 51: unconnected-(J1-Pad51) -> /FB2.MFD.N
- J1 pad 52: unconnected-(J1-Pad52) -> /FB3.LS3
- J1 pad 53: unconnected-(J1-Pad53) -> /FB2.MFD.P
- J1 pad 54: unconnected-(J1-Pad54) -> /FB3.HS3
- J1 pad 55: unconnected-(J1-Pad55) -> /FB2.MFDCLK.N
- J1 pad 57: unconnected-(J1-Pad57) -> /FB2.MFDCLK.P
- J1 pad 59: unconnected-(J1-Pad59) -> /FB2.LS5
- J1 pad 61: unconnected-(J1-Pad61) -> /FB2.HS5
- J1 pad 62: unconnected-(J1-Pad62) -> /FB3.HS2
- J1 pad 63: unconnected-(J1-Pad63) -> /FB2.HF5
- J1 pad 64: unconnected-(J1-Pad64) -> /FB3.LS2
- J1 pad 65: unconnected-(J1-Pad65) -> /FB2.PREF.LS
- J1 pad 67: unconnected-(J1-Pad67) -> /FB2.PREF.HS
- J1 pad 69: /FB2.HF5 -> /FB2.PREF.G
- J1 pad 72: unconnected-(J1-Pad72) -> /FB3.DVML.MUX
- J1 pad 75: unconnected-(J1-Pad75) -> /FB2.HS6
- J1 pad 76: unconnected-(J1-Pad76) -> /FB3.LS1
- J1 pad 77: unconnected-(J1-Pad77) -> /FB2.LS6
- J1 pad 78: unconnected-(J1-Pad78) -> /FB3.HS1
- J2 pad 01: unconnected-(J2-Pad01) -> /FB1.HF1
- J2 pad 02: unconnected-(J2-Pad02) -> /FB4.LF
- J2 pad 03: unconnected-(J2-Pad03) -> /FB1.HS1
- J2 pad 04: unconnected-(J2-Pad04) -> /FB4.LS6
- J2 pad 05: unconnected-(J2-Pad05) -> /FB1.LS1
- J2 pad 06: unconnected-(J2-Pad06) -> /FB4.HS6
- J2 pad 07: unconnected-(J2-Pad07) -> /FB1.LF
- J2 pad 08: unconnected-(J2-Pad08) -> /FB4.HF6
- J2 pad 09: unconnected-(J2-Pad09) -> /FB1.DVML.MUX
- J2 pad 10: unconnected-(J2-Pad10) -> /FB4.PREF.F
- J2 pad 11: unconnected-(J2-Pad11) -> /FB1.DVMH
- J2 pad 12: unconnected-(J2-Pad12) -> /FB4.PREF.G
- J2 pad 13: unconnected-(J2-Pad13) -> /FB1.DVML
- J2 pad 14: unconnected-(J2-Pad14) -> /FB4.PREF.HS
- J2 pad 15: unconnected-(J2-Pad15) -> /FB1.LF
- J2 pad 16: unconnected-(J2-Pad16) -> /FB4.PREF.LS
- J2 pad 17: unconnected-(J2-Pad17) -> /FB1.LS2
- J2 pad 18: unconnected-(J2-Pad18) -> /FB4.HF5
- J2 pad 19: unconnected-(J2-Pad19) -> /FB1.HS2
- J2 pad 20: unconnected-(J2-Pad20) -> /FB4.HS5
- J2 pad 21: unconnected-(J2-Pad21) -> /FB1.HF2
- J2 pad 22: unconnected-(J2-Pad22) -> /FB4.LS5
- J2 pad 23: unconnected-(J2-Pad23) -> /FB1.LF
- J2 pad 24: unconnected-(J2-Pad24) -> /FB4.MFDCLK.P
- J2 pad 25: unconnected-(J2-Pad25) -> /FB1.HF3
- J2 pad 26: unconnected-(J2-Pad26) -> /FB4.MFDCLK.N
- J2 pad 27: unconnected-(J2-Pad27) -> /FB1.HS3
- J2 pad 28: unconnected-(J2-Pad28) -> /FB4.MFD.P
- J2 pad 29: unconnected-(J2-Pad29) -> /FB1.LS3
- J2 pad 30: unconnected-(J2-Pad30) -> /FB4.MFD.N
- J2 pad 31: unconnected-(J2-Pad31) -> /FB1.LF
- J2 pad 32: unconnected-(J2-Pad32) -> /FB4.LF
- J2 pad 33: unconnected-(J2-Pad33) -> /FB1.MLD.N
- J2 pad 34: unconnected-(J2-Pad34) -> /FB4.LS4
- J2 pad 35: unconnected-(J2-Pad35) -> /FB1.MLD.P
- J2 pad 36: unconnected-(J2-Pad36) -> /FB4.HS4
- J2 pad 37: unconnected-(J2-Pad37) -> /FB1.MLDCLK.N
- J2 pad 38: unconnected-(J2-Pad38) -> /FB4.HF4
- J2 pad 39: unconnected-(J2-Pad39) -> /FB1.MLDCLK.P
- J2 pad 40: unconnected-(J2-Pad40) -> /FB4.LF
- J2 pad 41: unconnected-(J2-Pad41) -> /FB1.LF
- J2 pad 42: unconnected-(J2-Pad42) -> /FB4.MLDCLK.P
- J2 pad 43: unconnected-(J2-Pad43) -> /FB1.HF4
- J2 pad 44: unconnected-(J2-Pad44) -> /FB4.MLDCLK.N
- J2 pad 45: unconnected-(J2-Pad45) -> /FB1.HS4
- J2 pad 46: unconnected-(J2-Pad46) -> /FB4.MLD.P
- J2 pad 47: unconnected-(J2-Pad47) -> /FB1.LS4
- J2 pad 48: unconnected-(J2-Pad48) -> /FB4.MLD.N
- J2 pad 49: unconnected-(J2-Pad49) -> /FB1.LF
- J2 pad 50: unconnected-(J2-Pad50) -> /FB4.LF
- J2 pad 51: unconnected-(J2-Pad51) -> /FB1.MFD.N
- J2 pad 52: unconnected-(J2-Pad52) -> /FB4.LS3
- J2 pad 53: unconnected-(J2-Pad53) -> /FB1.MFD.P
- J2 pad 54: unconnected-(J2-Pad54) -> /FB4.HS3
- J2 pad 55: unconnected-(J2-Pad55) -> /FB1.MFDCLK.N
- J2 pad 56: unconnected-(J2-Pad56) -> /FB4.HF3
- J2 pad 57: unconnected-(J2-Pad57) -> /FB1.MFDCLK.P
- J2 pad 58: unconnected-(J2-Pad58) -> /FB4.LF
- J2 pad 59: unconnected-(J2-Pad59) -> /FB1.LS5
- J2 pad 60: unconnected-(J2-Pad60) -> /FB4.HF2
- J2 pad 61: unconnected-(J2-Pad61) -> /FB1.HS5
- J2 pad 62: unconnected-(J2-Pad62) -> /FB4.HS2
- J2 pad 63: unconnected-(J2-Pad63) -> /FB1.HF5
- J2 pad 64: unconnected-(J2-Pad64) -> /FB4.LS2
- J2 pad 65: unconnected-(J2-Pad65) -> /FB1.PREF.LS
- J2 pad 66: unconnected-(J2-Pad66) -> /FB4.LF
- J2 pad 67: unconnected-(J2-Pad67) -> /FB1.PREF.HS
- J2 pad 68: unconnected-(J2-Pad68) -> /FB4.DVML
- J2 pad 69: unconnected-(J2-Pad69) -> /FB1.PREF.G
- J2 pad 70: unconnected-(J2-Pad70) -> /FB4.DVMH
- J2 pad 71: unconnected-(J2-Pad71) -> /FB1.PREF.F
- J2 pad 72: unconnected-(J2-Pad72) -> /FB4.DVML.MUX
- J2 pad 73: unconnected-(J2-Pad73) -> /FB1.HF6
- J2 pad 74: unconnected-(J2-Pad74) -> /FB4.LF
- J2 pad 75: unconnected-(J2-Pad75) -> /FB1.HS6
- J2 pad 76: unconnected-(J2-Pad76) -> /FB4.LS1
- J2 pad 77: unconnected-(J2-Pad77) -> /FB1.LS6
- J2 pad 78: unconnected-(J2-Pad78) -> /FB4.HS1
- J2 pad 79: unconnected-(J2-Pad79) -> /FB1.LF
- J2 pad 80: unconnected-(J2-Pad80) -> /FB4.HF1
- J3 pad A46: unconnected-(U1-PadA46) -> /FB4.HF1
- J3 pad A48: unconnected-(U1-PadA48) -> /FB4.DVMH
- J3 pad A50: unconnected-(U1-PadA50) -> /FB4.DVML
- J3 pad A52: unconnected-(U1-PadA52) -> /FB4.LF
- J3 pad A54: unconnected-(U1-PadA54) -> /FB4.HF2
- J3 pad A59: unconnected-(U1-PadA59) -> /FB4.HF3
- J3 pad A61: unconnected-(U1-PadA61) -> /FB4.LF
- J3 pad A62: unconnected-(U1-PadA62) -> /FB4.MLD.N
- J3 pad A63: unconnected-(U1-PadA63) -> /FB4.LF
- J3 pad A64: unconnected-(U1-PadA64) -> /FB4.MLDCLK.N
- J3 pad A65: unconnected-(U1-PadA65) -> /FB4.LF
- J3 pad A68: unconnected-(U1-PadA68) -> /FB4.HF4
- J3 pad A70: unconnected-(U1-PadA70) -> /FB4.LF
- J3 pad A71: unconnected-(U1-PadA71) -> /FB4.MFD.N
- J3 pad A72: unconnected-(U1-PadA72) -> /FB4.LF
- J3 pad A73: unconnected-(U1-PadA73) -> /FB4.MFDCLK.N
- J3 pad A74: unconnected-(U1-PadA74) -> /FB4.LF
- J3 pad A76: unconnected-(U1-PadA76) -> /FB4.HF5
- J3 pad A79: unconnected-(U1-PadA79) -> /FB4.LF
- J3 pad A80: unconnected-(U1-PadA80) -> /FB4.PREF.HS
- J3 pad A81: unconnected-(U1-PadA81) -> /FB4.LF
- J3 pad A82: unconnected-(U1-PadA82) -> /FB4.PREF.F
- J3 pad A83: unconnected-(U1-PadA83) -> /FB4.LF
- J3 pad A85: unconnected-(U1-PadA85) -> /FB4.HF6
- J3 pad A87: unconnected-(U1-PadA87) -> /FB4.LF
- J3 pad B1: unconnected-(U1-PadB1) -> /FB3.HS1
- J3 pad B14: unconnected-(U1-PadB14) -> /FB3.HS3
- J3 pad B16: unconnected-(U1-PadB16) -> /FB3.LF
- J3 pad B17: unconnected-(U1-PadB17) -> /FB3.MLD.P
- J3 pad B18: unconnected-(U1-PadB18) -> /FB3.LF
- J3 pad B19: unconnected-(U1-PadB19) -> /FB3.MLDCLK.P
- J3 pad B20: unconnected-(U1-PadB20) -> /FB3.LF
- J3 pad B23: unconnected-(U1-PadB23) -> /FB3.HS4
- J3 pad B25: unconnected-(U1-PadB25) -> /FB3.LF
- J3 pad B26: unconnected-(U1-PadB26) -> /FB3.MFD.P
- J3 pad B27: unconnected-(U1-PadB27) -> /FB3.LF
- J3 pad B28: unconnected-(U1-PadB28) -> /FB3.MFDCLK.P
- J3 pad B29: unconnected-(U1-PadB29) -> /FB3.LF
- J3 pad B31: unconnected-(U1-PadB31) -> /FB3.HS5
- J3 pad B34: unconnected-(U1-PadB34) -> /FB3.LF
- J3 pad B35: unconnected-(U1-PadB35) -> /FB3.PREF.LS
- J3 pad B36: unconnected-(U1-PadB36) -> /FB3.LF
- J3 pad B40: unconnected-(U1-PadB40) -> /FB3.HS6
- J3 pad B42: unconnected-(U1-PadB42) -> /FB3.LF
- J3 pad B46: unconnected-(U1-PadB46) -> /FB4.HS1
- J3 pad B52: unconnected-(U1-PadB52) -> /FB4.LF
- J3 pad B54: unconnected-(U1-PadB54) -> /FB4.HS2
- J3 pad B59: unconnected-(U1-PadB59) -> /FB4.HS3
- J3 pad B61: unconnected-(U1-PadB61) -> /FB4.LF
- J3 pad B62: unconnected-(U1-PadB62) -> /FB4.MLD.P
- J3 pad B63: unconnected-(U1-PadB63) -> /FB4.LF
- J3 pad B64: unconnected-(U1-PadB64) -> /FB4.MLDCLK.P
- J3 pad B65: unconnected-(U1-PadB65) -> /FB4.LF
- J3 pad B68: unconnected-(U1-PadB68) -> /FB4.HS4
- J3 pad B70: unconnected-(U1-PadB70) -> /FB4.LF
- J3 pad B71: unconnected-(U1-PadB71) -> /FB4.MFD.P
- J3 pad B72: unconnected-(U1-PadB72) -> /FB4.LF
- J3 pad B73: unconnected-(U1-PadB73) -> /FB4.MFDCLK.P
- J3 pad B74: unconnected-(U1-PadB74) -> /FB4.LF
- J3 pad B76: unconnected-(U1-PadB76) -> /FB4.HS5
- J3 pad B79: unconnected-(U1-PadB79) -> /FB4.LF
- J3 pad B80: unconnected-(U1-PadB80) -> /FB4.PREF.LS
- J3 pad B85: unconnected-(U1-PadB85) -> /FB4.HS6
- J3 pad B87: unconnected-(U1-PadB87) -> /FB4.LF
- J3 pad B9: unconnected-(U1-PadB9) -> /FB3.HS2
- J3 pad C16: unconnected-(U1-PadC16) -> /FB3.LS3
- J3 pad C25: unconnected-(U1-PadC25) -> /FB3.LS4
- J3 pad C29: unconnected-(U1-PadC29) -> /FB3.LS5
- J3 pad C3: unconnected-(U1-PadC3) -> /FB3.LS1
- J3 pad C42: unconnected-(U1-PadC42) -> /FB3.LS6
- J3 pad C48: unconnected-(U1-PadC48) -> /FB4.LS1
- J3 pad C52: unconnected-(U1-PadC52) -> /FB4.LS2
- J3 pad C61: unconnected-(U1-PadC61) -> /FB4.LS3
- J3 pad C70: unconnected-(U1-PadC70) -> /FB4.LS4
- J3 pad C74: unconnected-(U1-PadC74) -> /FB4.LS5
- J3 pad C87: unconnected-(U1-PadC87) -> /FB4.LS6
- J3 pad E1: unconnected-(U1-PadE1) -> /FB2.LS6
- J3 pad E14: unconnected-(U1-PadE14) -> /FB2.LS5
- J3 pad E18: unconnected-(U1-PadE18) -> /FB2.LS4
- J3 pad E27: unconnected-(U1-PadE27) -> /FB2.LS3
- J3 pad E36: unconnected-(U1-PadE36) -> /FB2.LS2
- J3 pad E38: unconnected-(U1-PadE38) -> /FB2.DVML.MUX
- J3 pad E40: unconnected-(U1-PadE40) -> /FB2.LS1
- J3 pad E46: unconnected-(U1-PadE46) -> /FB1.LS6
- J3 pad E59: unconnected-(U1-PadE59) -> /FB1.LS5
- J3 pad E63: unconnected-(U1-PadE63) -> /FB1.LS4
- J3 pad E72: unconnected-(U1-PadE72) -> /FB1.LS3
- J3 pad E81: unconnected-(U1-PadE81) -> /FB1.LS2
- J3 pad E83: unconnected-(U1-PadE83) -> /FB1.DVML.MUX
- J3 pad E85: unconnected-(U1-PadE85) -> /FB1.LS1
- J3 pad F1: unconnected-(U1-PadF1) -> /FB2.LF
- J3 pad F12: unconnected-(U1-PadF12) -> /FB2.HS5
- J3 pad F14: unconnected-(U1-PadF14) -> /FB2.LF
- J3 pad F15: unconnected-(U1-PadF15) -> /FB2.MFDCLK.P
- J3 pad F16: unconnected-(U1-PadF16) -> /FB2.LF
- J3 pad F17: unconnected-(U1-PadF17) -> /FB2.MFD.P
- J3 pad F18: unconnected-(U1-PadF18) -> /FB2.LF
- J3 pad F20: unconnected-(U1-PadF20) -> /FB2.HS4
- J3 pad F23: unconnected-(U1-PadF23) -> /FB2.LF
- J3 pad F24: unconnected-(U1-PadF24) -> /FB2.MLDCLK.P
- J3 pad F25: unconnected-(U1-PadF25) -> /FB2.LF
- J3 pad F26: unconnected-(U1-PadF26) -> /FB2.MLD.P
- J3 pad F27: unconnected-(U1-PadF27) -> /FB2.LF
- J3 pad F29: unconnected-(U1-PadF29) -> /FB2.HS3
- J3 pad F3: unconnected-(U1-PadF3) -> /FB2.HS6
- J3 pad F34: unconnected-(U1-PadF34) -> /FB2.HS2
- J3 pad F36: unconnected-(U1-PadF36) -> /FB2.LF
- J3 pad F42: unconnected-(U1-PadF42) -> /FB2.HS1
- J3 pad F46: unconnected-(U1-PadF46) -> /FB1.LF
- J3 pad F48: unconnected-(U1-PadF48) -> /FB1.HS6
- J3 pad F5: unconnected-(U1-PadF5) -> /FB2.LF
- J3 pad F50: unconnected-(U1-PadF50) -> /FB1.LF
- J3 pad F51: unconnected-(U1-PadF51) -> /FB1.PREF.G
- J3 pad F52: unconnected-(U1-PadF52) -> /FB1.LF
- J3 pad F53: unconnected-(U1-PadF53) -> /FB1.PREF.LS
- J3 pad F54: unconnected-(U1-PadF54) -> /FB1.LF
- J3 pad F57: unconnected-(U1-PadF57) -> /FB1.HS5
- J3 pad F59: unconnected-(U1-PadF59) -> /FB1.LF
- J3 pad F6: unconnected-(U1-PadF6) -> /FB2.PREF.G
- J3 pad F60: unconnected-(U1-PadF60) -> /FB1.MFDCLK.P
- J3 pad F61: unconnected-(U1-PadF61) -> /FB1.LF
- J3 pad F62: unconnected-(U1-PadF62) -> /FB1.MFD.P
- J3 pad F63: unconnected-(U1-PadF63) -> /FB1.LF
- J3 pad F65: unconnected-(U1-PadF65) -> /FB1.HS4
- J3 pad F68: unconnected-(U1-PadF68) -> /FB1.LF
- J3 pad F69: unconnected-(U1-PadF69) -> /FB1.MLDCLK.P
- J3 pad F7: unconnected-(U1-PadF7) -> /FB2.LF
- J3 pad F70: unconnected-(U1-PadF70) -> /FB1.LF
- J3 pad F71: unconnected-(U1-PadF71) -> /FB1.MLD.P
- J3 pad F72: unconnected-(U1-PadF72) -> /FB1.LF
- J3 pad F74: unconnected-(U1-PadF74) -> /FB1.HS3
- J3 pad F79: unconnected-(U1-PadF79) -> /FB1.HS2
- J3 pad F8: unconnected-(U1-PadF8) -> /FB2.PREF.LS
- J3 pad F81: unconnected-(U1-PadF81) -> /FB1.LF
- J3 pad F87: unconnected-(U1-PadF87) -> /FB1.HS1
- J3 pad F9: unconnected-(U1-PadF9) -> /FB2.LF
- J3 pad G46: unconnected-(U1-PadG46) -> /FB1.LF
- J3 pad G48: unconnected-(U1-PadG48) -> /FB1.HF6
- J3 pad G50: unconnected-(U1-PadG50) -> /FB1.LF
- J3 pad G51: unconnected-(U1-PadG51) -> /FB1.PREF.F
- J3 pad G52: unconnected-(U1-PadG52) -> /FB1.LF
- J3 pad G53: unconnected-(U1-PadG53) -> /FB1.PREF.HS
- J3 pad G54: unconnected-(U1-PadG54) -> /FB1.LF
- J3 pad G57: unconnected-(U1-PadG57) -> /FB1.HF5
- J3 pad G59: unconnected-(U1-PadG59) -> /FB1.LF
- J3 pad G60: unconnected-(U1-PadG60) -> /FB1.MFDCLK.N
- J3 pad G61: unconnected-(U1-PadG61) -> /FB1.LF
- J3 pad G62: unconnected-(U1-PadG62) -> /FB1.MFD.N
- J3 pad G63: unconnected-(U1-PadG63) -> /FB1.LF
- J3 pad G65: unconnected-(U1-PadG65) -> /FB1.HF4
- J3 pad G68: unconnected-(U1-PadG68) -> /FB1.LF
- J3 pad G69: unconnected-(U1-PadG69) -> /FB1.MLDCLK.N
- J3 pad G70: unconnected-(U1-PadG70) -> /FB1.LF
- J3 pad G71: unconnected-(U1-PadG71) -> /FB1.MLD.N
- J3 pad G72: unconnected-(U1-PadG72) -> /FB1.LF
- J3 pad G74: unconnected-(U1-PadG74) -> /FB1.HF3
- J3 pad G79: unconnected-(U1-PadG79) -> /FB1.HF2
- J3 pad G81: unconnected-(U1-PadG81) -> /FB1.LF
- J3 pad G83: unconnected-(U1-PadG83) -> /FB1.DVML
- J3 pad G85: unconnected-(U1-PadG85) -> /FB1.DVMH
- J3 pad G87: unconnected-(U1-PadG87) -> /FB1.HF1
Routing:
- net /FB2.DVMH: track 18.8 -> 0.00 mm, vias 2 -> 1
- net /FB3.PREF.F: track 23.7 -> 10.8 mm, vias 1 -> 2
- net /FB2.DVML: track 12.2 -> 0.00 mm
- net /FB2.HF6: track 12.0 -> 0.00 mm
- net /FB3.HF6: track 0.00 -> 11.6 mm, vias 0 -> 2
- net /FB3.HF2: track 0.00 -> 10.0 mm, vias 0 -> 2
- net /FB3.LS6: track 0.00 -> 9.57 mm, vias 0 -> 1
- net /FB3.HS1: track 0.00 -> 9.37 mm, vias 0 -> 1
- net /FB3.HF1: track 0.00 -> 9.36 mm, vias 0 -> 1
- net /FB3.DVML: track 0.00 -> 8.57 mm, vias 0 -> 2
- net /FB3.HS6: track 0.00 -> 8.41 mm, vias 0 -> 1
- net /FB3.LS1: track 0.00 -> 8.19 mm, vias 0 -> 1
- net /FB3.LS2: track 0.00 -> 8.14 mm, vias 0 -> 2
- net /FB3.DVML.MUX: track 0.00 -> 8.04 mm, vias 0 -> 2
- net /FB3.HF5: track 0.00 -> 7.72 mm, vias 0 -> 1
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- added copper zone on In1.Cu, net /FB3.LF
- added copper zone on In2.Cu, net /FB3.LF
Other:
- board size 9.5 x 102.4 mm -> 9.5 x 102.6 mm
- copper layers 2 -> 4

Commit message: new route
Routing:
- net /FB2.HF6: track 0.00 -> 11.0 mm, vias 1 -> 2
- net /FB2.LS6: track 0.00 -> 8.91 mm
- net /FB2.HS6: track 0.00 -> 7.77 mm
- net /FB2.PREF.G: track 0.00 -> 7.25 mm, vias 1 -> 2
- net /FB2.PREF.LS: track 0.00 -> 6.77 mm, vias 1 -> 2
- net /FB2.PREF.HS: track 0.00 -> 6.57 mm, vias 1 -> 2
- net /FB2.LF: track 0.00 -> 6.24 mm, vias 18 -> 14
- net /FB2.PREF.F: track 0.00 -> 5.45 mm, vias 1 -> 2
- net /FB2.HS5: track 0.00 -> 2.77 mm, vias 1 -> 2
- net /FB2.MFD.P: track 0.00 -> 2.00 mm, vias 1 -> 2
- net /FB2.HF5: track 0.00 -> 1.91 mm, vias 1 -> 2
- net /FB2.MFDCLK.N: track 0.00 -> 1.80 mm, vias 1 -> 2
- net /FB2.LS5: track 0.00 -> 1.70 mm
- net /FB2.MFDCLK.P: track 0.00 -> 1.46 mm, vias 1 -> 2
- net /FB2.MFD.N: vias 1 -> 0
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
Commit message: routing update
Routing:
- net /FB2.HF1: track 0.00 -> 10.8 mm
- net /FB2.DVMH: track 0.00 -> 10.3 mm, vias 1 -> 3
- net /FB2.DVML: track 0.00 -> 9.06 mm, vias 1 -> 3
- net /FB2.HS1: track 0.00 -> 8.71 mm, vias 1 -> 3
- net /FB2.LS1: track 0.00 -> 7.89 mm, vias 1 -> 3
- net /FB2.LS2: track 0.00 -> 7.71 mm
- net /FB2.DVML.MUX: track 0.00 -> 7.31 mm
- net /FB2.HS2: track 0.00 -> 7.29 mm
- net /FB2.HF2: track 0.00 -> 7.27 mm, vias 1 -> 3
- net /FB2.LF: track 6.24 -> 13.1 mm, vias 14 -> 21
- net /FB2.MLD.N: track 0.00 -> 5.15 mm, vias 1 -> 3
- net /FB2.HF4: track 0.00 -> 4.94 mm
- net /FB2.HS4: track 0.00 -> 4.76 mm
- net /FB2.HS3: track 0.00 -> 3.84 mm, vias 1 -> 3
- net /FB2.MLD.P: track 0.00 -> 3.41 mm, vias 1 -> 3
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- added copper zone on In1.Cu, net /FB2.LF
- added copper zone on In2.Cu, net /FB2.LF

Commit message: more routing
Routing:
- net /FB3.LF: track 12.3 -> 12.2 mm, vias 18 -> 27
- net /FB2.LF: vias 21 -> 22
Changed lines of the file:
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@@
 	)
 	(via
-		(at 74.5066 86.5564)
+		(at 74.5236 86.614)
 		(size 0.5588)
 		(drill 0.254)
@@
 	)
 	(segment
+		(start 74.868021 79.970597)
+		(end 75.158719 79.970597)
+		(width 0.127)
+		(layer "In2.Cu")
+		(net 20)
+	)
+	(segment
+		(start 74.5236 86.614)
+		(end 74.041 86.1314)
+		(width 0.127)
+		(layer "In2.Cu")
+		(net 20)
+	)
+	(segment
+		(start 74.041 86.1314)
+		(end 74.041 80.797618)
+		(width 0.127)
+		(layer "In2.Cu")
+		(net 20)
+	)
+	(segment
 		(start 74.041 80.797618)
-		(end 74.041 86.0908)
-		(width 0.127)
-		(layer "In2.Cu")
-		(net 20)
-	)
-	(segment
-		(start 74.041 86.0908)
-		(end 74.5066 86.5564)
-		(width 0.127)
-		(layer "In2.Cu")
-		(net 20)
-	)
-	(segment
-		(start 75.158719 79.970597)
 		(end 74.868021 79.970597)
-		(width 0.127)
-		(layer "In2.Cu")
-		(net 20)
-	)
-	(segment
-		(start 74.868021 79.970597)
-		(end 74.041 80.797618)
 		(width 0.127)
 		(layer "In2.Cu")
@@
 	)
 	(via blind
-		(at 70.1294 59.7916)
+		(at 69.964146 69.980048)
+		(size 0.5588)
+		(drill 0.254)
+		(layers "In1.Cu" "In2.Cu")
+		(net 395)
+	)
+	(via blind
+		(at 69.964146 49.863248)
+		(size 0.5588)
+		(drill 0.254)
+		(layers "In1.Cu" "In2.Cu")
+		(net 395)
+	)
+	(via blind
+		(at 69.989546 72.215248)
+		(size 0.5588)
+		(drill 0.254)
+		(layers "In1.Cu" "In2.Cu")
+		(net 395)
+	)
+	(via blind
+		(at 70.1058 62.0141)
 		(size 0.5588)
 		(drill 0.254)
@@
 	)
 	(via blind
-		(at 70.1058 74.3077)
-		(size 0.5588)
-		(drill 0.254)
-		(layers "In1.Cu" "B.Cu")
-		(net 395)
-	)
-	(via blind
-		(at 70.1058 79.8957)
-		(size 0.5588)
-		(drill 0.254)
-		(layers "In1.Cu" "B.Cu")
-		(net 395)
-	)
-	(via blind
-		(at 70.1058 64.2493)
-		(size 0.5588)
-		(drill 0.254)
-		(layers "In1.Cu" "B.Cu")
-		(net 395)
-	)
-	(via blind
-		(at 70.1058 72.0725)
-		(size 0.5588)
-		(drill 0.254)
-		(layers "In1.Cu" "B.Cu")
-		(net 395)
-	)
-	(via blind
-		(at 70.1058 62.0141)
-		(size 0.5588)
-		(drill 0.254)
-		(layers "In1.Cu" "B.Cu")
-		(net 395)
-	)
-	(via blind
-		(at 70.1058 69.8373)
-		(size 0.5588)
-		(drill 0.254)
-		(layers "In1.Cu" "B.Cu")
-		(net 395)
-	)
-	(via blind
-		(at 70.1058 49.7205)
-		(size 0.5588)
-		(drill 0.254)
-		(layers "In1.Cu" "B.Cu")
-		(net 395)
-	)
-	(via blind
-		(at 70.104 84.3534)
-		(size 0.5588)
-		(drill 0.254)
-		(layers "In1.Cu" "B.Cu")
-		(net 395)
-	)
-	(via blind
-		(at 70.104 82.1436)
-		(size 0.5588)
-		(drill 0.254)
-		(layers "In1.Cu" "B.Cu")
+		(at 70.014946 64.417448)
+		(size 0.5588)
+		(drill 0.254)
+		(layers "In1.Cu" "In2.Cu")
+		(net 395)
+	)
+	(via blind
+		(at 69.989546 59.921648)
+		(size 0.5588)
+		(drill 0.254)
+		(layers "In1.Cu" "In2.Cu")
+		(net 395)
+	)
+	(via blind
+		(at 69.989546 74.450448)
+		(size 0.5588)
+		(drill 0.254)
+		(layers "In1.Cu" "In2.Cu")
+		(net 395)
+	)
+	(via blind
+		(at 69.989546 82.273648)
+		(size 0.5588)
+		(drill 0.254)
+		(layers "In1.Cu" "In2.Cu")
+		(net 395)
+	)
+	(via blind
+		(at 69.989546 80.038448)
+		(size 0.5588)
+		(drill 0.254)
+		(layers "In1.Cu" "In2.Cu")
+		(net 395)
+	)
+	(via blind
+		(at 69.937674 84.587033)
+		(size 0.5588)
+		(drill 0.254)
+		(layers "In1.Cu" "In2.Cu")
+		(net 395)
+	)
+	(via micro
+		(at 70.2564 49.4792)
+		(size 0.3556)
+		(drill 0.1524)
+		(layers "In2.Cu" "B.Cu")
+		(net 395)
+	)
+	(via micro
+		(at 70.2818 74.0664)
+		(size 0.3556)
+		(drill 0.1524)
+		(layers "In2.Cu" "B.Cu")
+		(net 395)
+	)
+	(via micro
+		(at 70.2818 59.5376)
+		(size 0.3556)
+		(drill 0.1524)
+		(layers "In2.Cu" "B.Cu")
+		(net 395)
+	)
+	(via micro
+		(at 70.3072 64.0334)
+		(size 0.3556)
+		(drill 0.1524)
+		(layers "In2.Cu" "B.Cu")
+		(net 395)
+	)
+	(via micro
+		(at 70.2564 69.596)
+		(size 0.3556)
+		(drill 0.1524)
+		(layers "In2.Cu" "B.Cu")
+		(net 395)
+	)
+	(via micro
+		(at 70.2818 81.8896)
+		(size 0.3556)
+		(drill 0.1524)
+		(layers "In2.Cu" "B.Cu")
+		(net 395)
+	)
+	(via micro
+		(at 70.229928 84.202985)
+		(size 0.3556)
+		(drill 0.1524)
+		(layers "In2.Cu" "B.Cu")
+		(net 395)
+	)
+	(via micro
+		(at 70.2818 71.8312)
+		(size 0.3556)
+		(drill 0.1524)
+		(layers "In2.Cu" "B.Cu")
+		(net 395)
+	)
+	(via micro
+		(at 70.2818 79.6544)
+		(size 0.3556)
+		(drill 0.1524)
+		(layers "In2.Cu" "B.Cu")
+		(net 395)
+	)
+	(segment
+		(start 70.229928 84.202985)
+		(end 70.393043 84.3661)
+		(width 0.254)
+		(layer "B.Cu")
 		(net 395)
 	)
@@
 	)
 	(segment
-		(start 71.2234 84.3661)
-		(end 70.1058 84.3661)
+		(start 70.393043 84.3661)
+		(end 71.2234 84.3661)
 		(width 0.254)
 		(layer "B.Cu")
@@
 	)
 	(segment
-		(start 73.253503 77.533499)
-		(end 73.253503 76.410328)
-		(width 0.254)
-		(layer "F.Cu")
-		(net 402)
-	)
-	(segment
-		(start 73.253503 76.410328)
+		(start 73.0885 76.245325)
 		(end 72.011875 75.1687)
 		(width 0.254)
@@
 		(net 402)
 	)
-	(via
-		(at 73.253503 77.533499)
-		(size 0.5588)
-		(drill 0.254)
-		(layers "F.Cu" "B.Cu")
+	(segment
+		(start 73.0885 77.532247)
+		(end 73.0885 76.245325)
+		(width 0.254)
+		(layer "F.Cu")
 		(net 402)
 	)
-	(segment
-		(start 73.253503 77.533499)
-		(end 70.6392 77.533499)
+	(via
+		(at 73.0885 77.532247)
+		(size 0.5588)
+		(drill 0.254)
+		(layers "F.Cu" "B.Cu")
+		(net 402)
+	)
+	(segment
+		(start 70.637948 77.532247)
+		(end 70.1058 77.000099)
+		(width 0.254)
+		(layer "B.Cu")
+		(net 402)
+	)
+	(segment
+		(start 73.0885 77.532247)
+		(end 70.637948 77.532247)
 		(width 0.254)
 		(layer "B.Cu")
@@
 	)
 	(segment
-		(start 70.6392 77.533499)
-		(end 70.1058 77.000099)
-		(width 0.254)
-		(layer "B.Cu")
-		(net 402)
-	)
-	(segment
 		(start 72.305217 66.3067)
 		(end 72.305217 66.875358)
@@
 	)
 	(via blind
-		(at 76.8096 82.1436)
+		(at 76.708 57.7596)
+		(size 0.5588)
+		(drill 0.254)
+		(layers "In1.Cu" "In2.Cu")
+		(free yes)
+		(net 405)
+	)
+	(via blind
+		(at 76.7334 62.1792)
+		(size 0.5588)
+		(drill 0.254)
+		(layers "In1.Cu" "In2.Cu")
+		(free yes)
+		(net 405)
+	)
+	(via blind
+		(at 76.8096 69.8754)
 		(size 0.5588)
 		(drill 0.254)
@@
 	)
 	(via blind
-		(at 76.708 57.7596)
+		(at 76.706068 82.376299)
 		(size 0.5588)
 		(drill 0.254)
@@
 	)
 	(via blind
-		(at 76.7334 62.1792)
+		(at 76.835 59.9948)
 		(size 0.5588)
 		(drill 0.254)
@@
 		(net 405)
 	)
-	(via blind
-		(at 76.8096 69.8754)
-		(size 0.5588)
-		(drill 0.254)
-		(layers "In1.Cu" "B.Cu")
+	(via micro
+		(at 76.941857 61.743941)
+		(size 0.3556)
+		(drill 0.1524)
+		(layers "In2.Cu" "B.Cu")
 		(net 405)
 	)
-	(via blind
-		(at 76.835 59.9948)
-		(size 0.5588)
-		(drill 0.254)
-		(layers "In1.Cu" "In2.Cu")
-		(free yes)
+	(via micro
+		(at 76.8114 67.6021)
+		(size 0.3556)
+		(drill 0.1524)
+		(layers "In2.Cu" "B.Cu")
 		(net 405)
 	)
 	(via micro
-		(at 76.941857 61.743941)
-		(size 0.3556)
-		(drill 0.1524)
-		(layers "In2.Cu" "B.Cu")
-		(net 405)
-	)
-	(via micro
-		(at 76.8114 67.6021)
-		(size 0.3556)
-		(drill 0.1524)
+		(at 76.916457 81.886141)
+		(size 0.3556)
+		(drill 0.1524)

Commit message: layout done
Routing:
- net /FB1.LF: track 0.00 -> 13.1 mm, vias 0 -> 24
- net /FB4.LF: track 0.00 -> 12.2 mm, vias 0 -> 28
- net /FB4.HF6: track 0.00 -> 11.6 mm, vias 0 -> 3
- net /FB1.HF6: track 0.00 -> 11.3 mm, vias 0 -> 3
- net /FB1.HF1: track 0.00 -> 10.8 mm, vias 0 -> 1
- net /FB4.PREF.F: track 0.00 -> 10.6 mm, vias 0 -> 2
- net /FB1.DVMH: track 0.00 -> 10.3 mm, vias 0 -> 3
- net /FB4.DVMH: track 0.00 -> 9.97 mm, vias 0 -> 2
- net /FB4.HS1: track 0.00 -> 9.88 mm, vias 0 -> 1
- net /FB4.HF2: track 0.00 -> 9.81 mm, vias 0 -> 1
- net /FB4.HF1: track 0.00 -> 9.78 mm, vias 0 -> 1
- net /FB4.LS6: track 0.00 -> 9.57 mm, vias 0 -> 1
- net /FB1.DVML: track 0.00 -> 9.06 mm, vias 0 -> 3
- net /FB4.DVML: track 0.00 -> 9.04 mm, vias 0 -> 3
- net /FB1.LS6: track 0.00 -> 8.91 mm, vias 0 -> 1
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- added copper zone on In1.Cu, net /FB1.LF
- added copper zone on In2.Cu, net /FB1.LF
- added copper zone on In1.Cu, net /FB4.LF
- added copper zone on In2.Cu, net /FB4.LF
Other:
- board text added: "NOTE C: ALL VIAS TO BE FILLED"
- board text added: "Note A: Slot Holes on the Edge from Secondary Side"
- board text added: "Note B: Counterbore from Primary Side"
- board text added: "SCALE: NONE NON- PLATED"
- board text removed: "Note A: Counterbore from Secondary Side"

Commit message: final design
Routing:
- net /FB3.HF4: track 4.68 -> 6.57 mm
- net /FB2.HF4: track 4.94 -> 6.71 mm
- net /FB4.HF5: track 7.27 -> 8.10 mm
- net /FB3.HF5: track 7.27 -> 8.03 mm
- net /FB3.HS2: track 7.63 -> 8.18 mm
- net /FB2.HS2: track 7.29 -> 7.80 mm
